Commit message: adiciona plugin kinematics e moveit_config

File: victory_description/urdf/victory.urdf (robot description, URDF)
Before this commit: robot elir_test, 5 links, 4 joints
Links:
- added link victory_ref
Joints:
- added joint joint_ref: type fixed, parent victory_link3, child victory_ref, origin xyz=0 0 0.3 rpy=0 0 0, axis 0 0 0
- joint joint_hand: axis 1 0 0 -> 0.1 0 0; parent victory_link3 -> victory_ref

File: victory_description/urdf/victory.urdf.xacro (robot description, xacro)
@@ -1,4 +1,4 @@
 <?xml version="1.0" ?>
-<robot name="elir_test" xmlns:xacro="http://www.ros.org/wiki/xacro">
+<robot name="victory" xmlns:xacro="http://www.ros.org/wiki/xacro">
 <xacro:property name="M_PI" value="3.141592" />
   <material name="purple">
@@ -102,5 +102,5 @@
     </collision>
     </link>
-    <!-- <joint name="joint_ref" type="fixed">
+    <joint name="joint_ref" type="fixed">
       <parent link="victory_link3"/>
       <child link="victory_ref"/>
@@ -108,10 +108,10 @@
       <axis xyz="0 0 0"/>
     </joint>
-    <link name="victory_ref"/> -->
+    <link name="victory_ref"/>
     <joint name="joint_hand" type="fixed">
-      <parent link="victory_link3"/>
+      <parent link="victory_ref"/>
       <child link="victory_hand"/>
       <origin rpy="0 0 0" xyz="0.0 0.0 0.0"/>
-      <axis xyz="1 0 0"/>
+      <axis xyz="0.1 0 0"/>
     </joint>
     <link name="victory_hand">
@@ -122,5 +122,5 @@
       </geometry>
       <material name="light_blue"/>
-      <origin rpy="0 0 0" xyz="0.015 0.0 ${0.6}"/>
+      <origin rpy="0 0 0" xyz="0.00 0.0 ${0.405}"/>
     </visual>
     <!-- this collision is for the front f1 claw unit -->
